File: Electronics/Oudini/FTIR_v0.1.sch (EAGLE design)
At the start: 93 parts, among them CON1 SPI, IC1 REG1117, J1 22--02, J2 22--02, J3 22--02, J7 22--02, Q1 IRF3704S, Q3 IRF3704S, Q4 BSP75, Q6 BSP75, Q7 IRF3704S, Q8 BSP75, X3 16MHz, X4 MINI-USB

Commit message: started electronic design of the main board
Parts:
- removed I/O3, I/O5: RJ12, lpatiny:RJ12STRAIGHT
- removed J1, J2, J3, J7: 22--02, lpatiny:22--02
- removed LED6, LED8: Blue, adafruit:LEDCHIPLED_1206
- removed Q6: BSP75, infineon:BSP613P
- removed R35, R7: 1k, rcl:R-EU_R0805
- added C13: 100nF, rcl:C-EUC1206
- added C14: 10uF, rcl:C-EUC1206
- added C15, C17: 0.22nF, rcl:C-EUC1206
- added C18: 4.7uF, rcl:C-EUC1206
- added PIEZO: RJ12, lpatiny:RJ12STRAIGHT
- added R4: 10k, rcl:R-EU_R0805
- added RL12: 1K, rcl:R-EU_R0805
- added RL13, RL14, RL15, RL16, RL17: 10K, rcl:R-EU_R0805
- added U$13: SZ05-ZIGBEESMD, lpatiny:SZ05-ZIGBEESMD
- added U$14: DAC1220, FTIR:DAC1220
- added U$15: MCP3425, phMeter:MCP3425
- added U$16, U$17, U$18, U$19: JACK_PJ-063BH, lpatiny:JACK_PJ-063BH
- U$3: value SZ05-ZIGBEE -> AMP_MATE_N_LOCK; device lpatiny:SZ05-ZIGBEETHROUGHHOLE -> lpatiny:AMP_MATE_N_LOCK
- U$6: value KPJX-4S-S -> JACK_PJ-063BH; device lpatiny:KPJX-4S-S -> lpatiny:JACK_PJ-063BH
- renumbered I/O2 to SENSOR
Connections:
- removed net D5: RL11.1
- removed net D6: RL10.1
- removed net N$19: I/O5.2, LED8.C, Q6.D@1
- removed net N$32: I/O5.3, R35.2
- removed net N$33: LED8.A, R7.1
- removed net N$36: J7-2.S, Q7.D
- removed net N$38: J3-2.S, Q8.D@1
- new net 2.5V: C17.2, U$14.VREF
- new net DGND: C13.1, C14.1, U$15.VSS
- new net N$29: C17.1, U$14.C1
- new net N$30: Q7.D, U$6.GND
- new net N$4: Q4.D@1, U$19.GND
- new net N$5: R4.1, R5.1, U$14.CS
- new net PIEZO: C15.2, PIEZO.3, U$14.VOUT
- net +12V: now also PIEZO.1, U$16.V+, U$17.V+, U$18.V+, U$19.V+, U$3.+12V, U$6.V+; no longer I/O3.1, I/O5.1, J1-1.S, J2-1.S, J3-1.S, J7-1.S, U$6.+12V
- net +5V: now also C13.2, C14.2, C18.2, PIEZO.5, R4.2, U$13.VCC, U$14.AVDD, U$14.DVDD, U$15.VDD, U$3.+5V; no longer I/O3.5, I/O5.5, R5.2, R7.2, U$3.VCC, U$6.+5V
- net A4: now also U$15.VIN+
- net AGND: now also U$14.AGND
- net D10*: now also RL1.1
- net D11*: no longer Q6.G
- net D5*: now also RL11.1
- net D6*: now also RL10.1
- net D7*: no longer RL1.1
- net D8*: now also R5.2; no longer R35.1
- net D9*: now also RL12.1; no longer Q4.G
- net GND: now also C18.1, PIEZO.4, PIEZO.6, RL13.1, RL14.1, RL15.1, RL16.1, RL17.1, U$13.GND, U$13.SGND, U$14.DGND, U$3.GND1, U$3.GND2; no longer I/O3.4, I/O3.6, I/O5.4, I/O5.6, Q6.S, U$3.GND, U$3.SGND, U$6.GND1, U$6.GND2
- net GND1: now also U$13.RNU; no longer U$3.RNU
- net GND2: now also U$13.NET; no longer U$3.NET
- net GND3: now also U$13.ALM; no longer U$3.ALM
- net MOSI: now also U$14.SDIO
- net N$1: now also Q4.G, RL12.2, RL17.2; no longer I/O3.2, LED6.C, Q4.D@1
- net N$11: now also U$13.RX1; no longer U$3.RX1
- net N$13: now also RL15.2
- net N$15: now also C15.1, U$14.C2; no longer J1-2.S, Q3.D
- net N$22: now also Q8.D@1, U$18.GND; no longer LED6.A, R5.1
- net N$24: now also U$13.TX1; no longer U$3.TX1
- net N$28: now also RL13.2
- net N$34: now also Q3.D, U$16.GND; no longer J2-2.S, Q1.D
- net N$35: now also U$13.CFG; no longer U$3.CFG
- net N$37: now also RL14.2
- net N$6: now also RL16.2
- net N$7: now also Q1.D, U$17.GND; no longer I/O3.3
- net SCK: now also U$14.SCLK
- net SCL: now also U$15.SCL
- net SDA: now also U$15.SDA
Other:
- note added: "12V pump"
- note added: "Peltier X2"
- note added: "Piezo driver"
- note added: "Power Supply 13A"
- note removed: "PZT driver"
- note removed: "Peletier X2"
- note removed: "Power"
- note removed: "RJ12"
- moved on the sheet: Q1, Q3, Q4, Q7, Q8, R5, RL1, RL10, RL11, RL2
