File: Electronics/Oudini/FTIR_v0.1.brd (EAGLE design)
At the start: 108.1 x 84.6 mm, 93 parts, among them CON1 SPI, IC1 REG1117, J1 22--02, J2 22--02, J3 22--02, J7 22--02, Q1 IRF3704S, Q3 IRF3704S, Q4 BSP75, Q6 BSP75, Q7 IRF3704S, Q8 BSP75, X3 16MHz, X4 MINI-USB

Commit message: started electronic design of the main board
Parts:
- removed I/O2, I/O3, I/O5: RJ12, lpatiny:RJ12-STRAIGHT
- removed J1, J2, J3, J7: 22--02, lpatiny:2-PIN-5.08S
- removed LED6, LED8: Blue, adafruit:CHIPLED_1206
- removed Q6: BSP75, infineon:PG-SOT-223
- removed R35, R7: 1k, rcl:R0805
- added C13: 100nF, rcl:C1206
- added C14: 10uF, rcl:C1206
- added C15, C17: 0.22nF, rcl:C1206
- added C18: 4.7uF, rcl:C1206
- added PIEZO, SENSOR: RJ12, lpatiny:RJ12-STRAIGHT
- added R4: 10k, rcl:R0805
- added RL12: 1K, rcl:R0805
- added RL13, RL14, RL15, RL16, RL17: 10K, rcl:R0805
- added U$13: SZ05-ZIGBEESMD, lpatiny:SZ05-ZIGBEE3
- added U$14: DAC1220, FTIR:SSOP-16
- added U$15: MCP3425, phMeter:SOT-23-6
- added U$16, U$17, U$18, U$19: JACK_PJ-063BH, lpatiny:PJ-063BH
- U$3: value SZ05-ZIGBEE -> AMP_MATE_N_LOCK; device lpatiny:SZ05-ZIGBEE4 -> lpatiny:AMP_MATE_N_LOCK
- U$6: value KPJX-4S-S -> JACK_PJ-063BH; device lpatiny:KPJX-4S-S -> lpatiny:PJ-063BH
- moved R5 275.6 mm to (1.27, -208.3), flipped to the top, turned to 0 degrees
- moved U$12 183.6 mm to (77.5, 68.6)
- moved U$11 165.3 mm to (77.5, 64.8), turned to 180 degrees
- moved U$10 158.5 mm to (77.5, 61.0), turned to 180 degrees
- moved Q8 156.1 mm to (15.6, 12.1), flipped to the bottom
- moved U$9 151.9 mm to (77.5, 57.1), turned to 180 degrees
- moved Q1 126.6 mm to (32.7, 13.3), flipped to the bottom, turned to 180 degrees
- moved RL2 88.9 mm to (80.0, 76.2)
- moved U$3 82.1 mm to (11.4, 29.2), turned to 0 degrees
- moved C5 77.3 mm to (88.9, 72.4)
- moved IC1 77.3 mm to (90.2, 63.5)
- moved C1 77.3 mm to (91.4, 69.8)
- moved Q3 77.2 mm to (68.6, 12.7), flipped to the bottom, turned to 180 degrees
- moved R28 54.1 mm to (42.5, 64.6)
- moved R29 53.4 mm to (46.5, 64.6)
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Connections:
- removed net D5: RL11.1
- removed net D6: RL10.1
- removed net N$19: I/O5.PWM, LED8.C, Q6.2
- removed net N$32: I/O5.I/O, R35.2
- removed net N$33: LED8.A, R7.1
- removed net N$36: J7.2, Q7.2
- removed net N$38: J3.2, Q8.2
- new net 2.5V: C17.2, U$14.VREF
- new net DGND: C13.1, C14.1, U$15.VSS
- new net N$29: C17.1, U$14.C1
- new net N$30: Q7.2, U$6.GND
- new net N$4: Q4.2, U$19.GND
- new net N$5: R4.1, R5.1, U$14.CS
- new net PIEZO: C15.2, PIEZO.I/O, U$14.VOUT
- net +12V: now also PIEZO.+12V, SENSOR.+12V, U$16.V+, U$17.V+, U$18.V+, U$19.V+, U$3.12V, U$6.V+; no longer I/O2.+12V, I/O3.+12V, I/O5.+12V, J1.1, J2.1, J3.1, J7.1, U$6.+12V
- net +5V: now also C13.2, C14.2, C18.2, PIEZO.+5V, R4.2, SENSOR.+5V, U$13.VCC, U$14.AVDD, U$14.DVDD, U$15.VDD, U$3.5V; no longer I/O2.+5V, I/O3.+5V, I/O5.+5V, R5.2, R7.2, U$3.VCC, U$6.+5V
- net A4: now also U$15.VIN+
- net AGND: now also U$14.AGND
- net D10*: now also RL1.1
- net D11*: no longer Q6.1
- net D5*: now also RL11.1
- net D6*: now also RL10.1
- net D7*: no longer RL1.1
- net D8*: now also R5.2; no longer R35.1
- net D9*: now also RL12.1; no longer Q4.1
- net GND: now also C18.1, PIEZO.GND1, PIEZO.GND2, RL13.1, RL14.1, RL15.1, RL16.1, RL17.1, SENSOR.GND1, SENSOR.GND2, U$13.GND, U$13.SND, U$14.DGND, U$3.GND1, U$3.GND2; no longer I/O2.GND1, I/O2.GND2, I/O3.GND1, I/O3.GND2, I/O5.GND1, I/O5.GND2, Q6.3, U$3.GND, U$3.SND, U$6.GND1, U$6.GND2
- net GND1: now also U$13.RUN; no longer U$3.RUN
- net GND2: now also U$13.NET; no longer U$3.NET
- net GND3: now also U$13.ALM; no longer U$3.ALM
- net MOSI: now also U$14.SDIO
- net N$1: now also Q4.1, RL12.2, RL17.2; no longer I/O3.PWM, LED6.C, Q4.2
- net N$11: now also U$13.RX1; no longer U$3.RX1
- net N$13: now also RL15.2
- net N$15: now also C15.1, U$14.C2; no longer J1.2, Q3.2
- net N$2: now also SENSOR.I/O; no longer I/O2.I/O
- net N$22: now also Q8.2, U$18.GND; no longer LED6.A, R5.1
- net N$24: now also U$13.TX1; no longer U$3.TX1
- net N$28: now also RL13.2
- net N$34: now also Q3.2, U$16.GND; no longer J2.2, Q1.2
- net N$35: now also U$13.CFG; no longer U$3.CFG
- net N$37: now also RL14.2
- net N$6: now also RL16.2
- net N$7: now also Q1.2, U$17.GND; no longer I/O3.I/O
- net SCK: now also U$14.SCLK
- net SCL: now also U$15.SCL
- net SDA: now also U$15.SDA
Routing:
- net +12V: track 384.5 -> 0.00 mm
- net +5V: track 299.0 -> 0.00 mm, vias 4 -> 0
- net GND: track 135.9 -> 0.00 mm, vias 8 -> 0
- net 3.3V: track 133.6 -> 0.00 mm
- net VUSB: track 63.4 -> 0.00 mm, vias 2 -> 0
- net +5V/1: track 54.3 -> 0.00 mm, vias 2 -> 0
- net USB_N: track 31.6 -> 0.00 mm
- net USB_P: track 31.6 -> 0.00 mm
- net N$19: track 29.6 -> 0.00 mm
- net N$1: track 29.4 -> 0.00 mm
- net AGND: track 28.8 -> 0.00 mm, vias 1 -> 0
- net USBC_P: track 25.2 -> 0.00 mm
- net USBC_N: track 25.2 -> 0.00 mm
- net N$36: track 12.8 -> 0.00 mm
- net N$2: track 12.4 -> 0.00 mm
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- added copper zone on layer 1, net +12V
- removed copper zone on layer 1, net GND
Other:
- board text removed: "5V"
- board text removed: "BioReactor"
- board text removed: "DAT"
- board text removed: "GND"
- board text removed: "IR Source"
- board text removed: "Integrated Bertha v1.1 Control Board"
- board text removed: "TX/RX"
- board text removed: "Tliquid"
- board text removed: "Tplate"

Commit message: main board Oudini on the way, 2.5V ref generator missing for the DAC stage, guard ring to be added on C1 C2 (see datasheet DAC1220)
Parts:
- removed R5: 1k, rcl:R0805
- added C20, C21: 18pF, rcl:C1206
- added QF1: ECS-10.7-7.5A, crystal:HC49U
- C15: value 0.22nF -> 2.2nF
- moved RL17 316.1 mm to (53.3, 71.8), flipped to the bottom, turned to 270 degrees
- moved RL16 263.1 mm to (48.9, 25.1), flipped to the bottom
- moved RL15 260.5 mm to (67.0, 24.8), flipped to the bottom
- moved C18 255.2 mm to (19.7, 59.1), flipped to the bottom
- moved C17 244.8 mm to (5.08, 55.6), flipped to the bottom, turned to 90 degrees
- moved RL13 241.8 mm to (30.8, 25.4), flipped to the bottom
- moved C15 239.8 mm to (8.89, 56.8), flipped to the bottom, turned to 90 degrees
- moved R4 235.5 mm to (30.5, 31.8), turned to 180 degrees
- moved RL14 235.1 mm to (20.6, 13.3), flipped to the bottom, turned to 270 degrees
- moved RL12 232.9 mm to (52.1, 59.7), flipped to the bottom, turned to 90 degrees
- moved U$14 232.4 mm to (15.2, 56.8), flipped to the bottom, turned to 270 degrees
- moved R9 183.8 mm to (74.9, 74.9)
- moved RL9 173.3 mm to (73.7, 69.8)
- moved RL7 164.5 mm to (83.8, 72.4)
- moved RL10 164.3 mm to (27.3, 26.4), flipped to the bottom, turned to 270 degrees
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Connections:
- removed net N$5: R4.1, R5.1, U$14.CS
- new net N$19: C21.1, QF1.3, U$14.XIN
- new net N$31: C20.1, QF1.1, U$14.XOUT
- net AGND: now also PIEZO.GND1, PIEZO.GND2, SENSOR.GND1, SENSOR.GND2
- net D8*: now also R4.1, U$14.CS; no longer R5.2
- net GND: now also C20.2, C21.2, QF1.2; no longer PIEZO.GND1, PIEZO.GND2, SENSOR.GND1, SENSOR.GND2
